File: checkpoint/checkpoint-pcb-v1.1/mcu.kicad_sch (KiCad schematic)
At the start: 30 parts, among them J11 BOOT, J12 Y_ENDSTOP, J13 SERVO, J14 RGB, J15 SWD, J19 I2C, Q1 BSS138, SW1 SW_RESET, U3 STM32G0B1CBTx, Y1 Crystal

Commit message: chore: reset refdes numbers
Parts:
- renumbered C18 to C16, C16 to C17, C19 to C18, C21 to C19, C17 to C20, C20 to C21, J19 to J11, J11 to J12, J12 to J13, J13 to J14, J14 to J15, J15 to J16, R23 to R22, R22 to R23, R27 to R26, R29 to R27, R26 to R28, R28 to R29

Commit message: fix: add i2c pullup resistors
Parts:
- added R22, R23: 4.7K, Resistor_SMD:R_0603_1608Metric, symbol Device:R
- renumbered J12 to J11, J13 to J12, J11 to J13, R22 to R24, R23 to R25, R24 to R26, R25 to R27, R26 to R28, R27 to R29, R28 to R30, R29 to R31, R30 to R32
Connections:
- net +3.3V: now also R22.1, R23.2
- net I2C_SCL: now also R22.2
- net I2C_SDA: now also R23.1
Other:
- moved on the sheet: J13

Commit message: chore: update component rotation
Parts:
- C14, C18, C19, C21, C22: value 0.1uF -> 100nF
Changed lines of the file:
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@@
 			)
 		)
-		(property "Value" "0.1uF"
+		(property "Value" "100nF"
 			(at 237.49 90.1699 0)
 			(effects
@@
 			)
 		)
-		(property "Value" "0.1uF"
+		(property "Value" "100nF"
 			(at 62.23 41.9099 0)
 			(effects
@@
 			)
 		)
-		(property "Value" "0.1uF"
+		(property "Value" "100nF"
 			(at 236.22 53.3399 0)
 			(effects
@@
 			)
 		)
-		(property "Value" "0.1uF"
+		(property "Value" "100nF"
 			(at 247.65 90.1699 0)
 			(effects
@@
 			)
 		)
-		(property "Value" "0.1uF"
+		(property "Value" "100nF"
 			(at 227.33 90.1699 0)
 			(effects
