File: checkpoint/KiCad/power.kicad_sch (KiCad schematic)
At the start: 21 parts, among them J18 PWR_OUT, J19 PWR_CAN_IN, U5 AMS1117-3.3, U6 TPS5430DDA

Commit message: fix: replace undersized protection diodes
Parts:
- D10: value SS34 -> SS54
- D11: value SS210 -> SS54
Changed lines of the file:
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@@
 			)
 		)
-		(property "Value" "SS210"
+		(property "Value" "SS54"
 			(at 154.94 88.5824 90)
 			(effects
@@
 			)
 		)
-		(property "Value" "SS34"
+		(property "Value" "SS54"
 			(at 99.06 74.93 0)
 			(effects
