File: ez-servo/KiCad/ez-servo.kicad_pcb (KiCad board)
At the start: 4 copper layers, 20 x 20 mm, 14 parts, among them J2 SERVO, J3 VSEL, U1 TPS5430DDA

Commit message: fix: add silkscreen markings
Routing:
- net VOUT: track 27.5 -> 30.8 mm, vias 0 -> 2
- net SERVO_PWM: track 23.2 -> 21.6 mm
- net SENSE: track 20.2 -> 20.4 mm, vias 1 -> 2
- net Net-(C2-Pad2): track 12.3 -> 12.4 mm, vias 1 -> 3
- net GND: vias 8 -> 2
Other:
- board text added: "6V"
- board text added: "8.4V"
- board text added: "EZServo ${REVISION}"
- board text added: "GND"
- board text added: "SIG"
- board text added: "VOL"
